Commit message: Update ROS bot model

File: ros/src/clumsybot_description/urdf/clumsybot.urdf (robot description, URDF)
Before this commit: robot clumsybot, 1 links, 0 joints
Links:
- added link hat_link; visual box size=0.15 0.2 0.04
- link base_link: geometry visual box size=0.145 0.19 0.25
Joints:
- added joint base_to_camera: type fixed, parent base_link, child hat_link, origin xyz=0 0 0.25

File: ros/src/clumsybot_description/urdf/clumsybot.xacro (robot description, xacro)
@@ -1,4 +1,4 @@
 <?xml version="1.0"?>
-<robot name="clumsybot">
+<robot name="clumsybotxacro">
   <xmlns:xacro="http://www.ros.org/wiki/xacro" name="clumsybot">
   <xacro:property name="base_width" value="0.19"/>
