Commit message: Use xacro for robot description

File: ros/src/clumsybot_description/urdf/clumsybot.urdf.xacro (robot description, xacro)
@@ -1,4 +1,9 @@
 <?xml version="1.0" ?>
 <robot name="clumsybot" xmlns:xacro="http://www.ros.org/wiki/xacro">
+  <xacro:property name="base_len" value="0.145"/>
+  <xacro:property name="base_width" value="0.19"/>
+  <xacro:property name="base_height" value="0.23"/>
+  <xacro:property name="hat_protuding" value="0.01"/>
+  <xacro:property name="hat_height" value="0.03"/>
   <material name="blue">
     <color rgba="0 0 0.8 1"/>
@@ -10,7 +15,7 @@
     <visual>
       <geometry>
-        <box size="0.145 0.19 0.25"/>
+        <box size="${base_len} ${base_width} ${base_height}"/>
       </geometry>
-      <origin xyz="0 0 0.125"/>
+      <origin xyz="0 0 ${base_height/2}"/>
       <material name="metalic"/>
     </visual>
@@ -19,5 +24,5 @@
     <visual>
       <geometry>
-        <box size="0.15 0.2 0.04"/>
+        <box size="${base_len+hat_protuding} ${base_width+hat_protuding} ${hat_height}"/>
       </geometry>
       <material name="blue"/>
@@ -27,5 +32,5 @@
     <parent link="base_link"/>
     <child link="hat_link"/>
-    <origin xyz="0 0 0.25"/>
+    <origin xyz="0 0 ${base_height}"/>
   </joint>
 </robot>

Commit message: Change ROS model and launch script to show Joint State Publisher with wheel rotation slider

File: ros/src/clumsybot_description/urdf/clumsybot.urdf.xacro (robot description, xacro)
@@ -1,4 +1,5 @@
 <?xml version="1.0" ?>
 <robot name="clumsybot" xmlns:xacro="http://www.ros.org/wiki/xacro">
+  <xacro:property name="PI" value="3.14159"/>
   <xacro:property name="base_len" value="0.145"/>
   <xacro:property name="base_width" value="0.19"/>
@@ -6,9 +7,15 @@
   <xacro:property name="hat_protuding" value="0.01"/>
   <xacro:property name="hat_height" value="0.03"/>
+  <xacro:property name="wheel_radius" value="0.021"/>
+  <xacro:property name="wheel_width" value="0.007"/>
+  <xacro:property name="wheel_clearance" value="0.005"/>
   <material name="blue">
     <color rgba="0 0 0.8 1"/>
   </material>
   <material name="metalic">
-    <color rgba="0.9 0.9 0.95 1"/>
+    <color rgba="0.8 0.8 0.9 1"/>
+  </material>
+  <material name="wheel_color">
+    <color rgba="0.1 0.1 0.1 1"/>
   </material>
   <link name="base_link">
@@ -17,5 +24,5 @@
         <box size="${base_len} ${base_width} ${base_height}"/>
       </geometry>
-      <origin xyz="0 0 ${base_height/2}"/>
+      <origin xyz="0 0 ${base_height/2}" rpy="0 0 0" />
       <material name="metalic"/>
     </visual>
@@ -29,8 +36,23 @@
     </visual>
   </link>
-  <joint name="base_to_camera" type="fixed">
+  <joint name="base_to_hat" type="fixed">
     <parent link="base_link"/>
     <child link="hat_link"/>
-    <origin xyz="0 0 ${base_height}"/>
+    <origin xyz="0 0 ${base_height}" />
+  </joint>
+  <link name="left_back_wheel">
+    <visual>
+      <geometry>
+        <cylinder length="${wheel_width}" radius="${wheel_radius}"/>
+      </geometry>
+      <material name="wheel_color"/>
+      <origin rpy="${PI/2} 0 0" />
+    </visual>
+  </link>
+  <joint name="left_back_wheel_joint" type="continuous">
+    <axis xyz="0 1 0"/>
+    <parent link="base_link"/>
+    <child link="left_back_wheel"/>
+    <origin xyz="${base_len/2 - wheel_radius} ${base_width/2} ${wheel_radius - wheel_clearance}"/>
   </joint>
 </robot>

Commit message: Add ROS definitions for wheels

File: ros/src/clumsybot_description/urdf/clumsybot.urdf.xacro (robot description, xacro)
@@ -41,4 +41,19 @@
     <origin xyz="0 0 ${base_height}" />
   </joint>
+  <link name="left_front_wheel">
+    <visual>
+      <geometry>
+        <cylinder length="${wheel_width}" radius="${wheel_radius}"/>
+      </geometry>
+      <material name="wheel_color"/>
+      <origin rpy="${PI/2} 0 0" />
+    </visual>
+  </link>
+  <joint name="left_front_wheel_joint" type="continuous">
+    <axis xyz="0 1 0"/>
+    <parent link="base_link"/>
+    <child link="left_front_wheel"/>
+    <origin xyz="${-base_len/2 + wheel_radius} ${base_width/2} ${wheel_radius - wheel_clearance}"/>
+  </joint>
   <link name="left_back_wheel">
     <visual>
@@ -51,4 +66,5 @@
   </link>
   <joint name="left_back_wheel_joint" type="continuous">
+    <mimic joint="left_front_wheel_joint" offset="0" multiplier="1" />
     <axis xyz="0 1 0"/>
     <parent link="base_link"/>
@@ -56,3 +72,34 @@
     <origin xyz="${base_len/2 - wheel_radius} ${base_width/2} ${wheel_radius - wheel_clearance}"/>
   </joint>
+  <link name="right_front_wheel">
+    <visual>
+      <geometry>
+        <cylinder length="${wheel_width}" radius="${wheel_radius}"/>
+      </geometry>
+      <material name="wheel_color"/>
+      <origin rpy="${PI/2} 0 0" />
+    </visual>
+  </link>
+  <joint name="right_front_wheel_joint" type="continuous">
+    <axis xyz="0 1 0"/>
+    <parent link="base_link"/>
+    <child link="right_front_wheel"/>
+    <origin xyz="${-base_len/2 + wheel_radius} ${-base_width/2} ${wheel_radius - wheel_clearance}"/>
+  </joint>
+  <link name="right_back_wheel">
+    <visual>
+      <geometry>
+        <cylinder length="${wheel_width}" radius="${wheel_radius}"/>
+      </geometry>
+      <material name="wheel_color"/>
+      <origin rpy="${PI/2} 0 0" />
+    </visual>
+  </link>
+  <joint name="right_back_wheel_joint" type="continuous">
+    <mimic joint="right_front_wheel_joint" offset="0" multiplier="1" />
+    <axis xyz="0 1 0"/>
+    <parent link="base_link"/>
+    <child link="right_back_wheel"/>
+    <origin xyz="${base_len/2 - wheel_radius} ${-base_width/2} ${wheel_radius - wheel_clearance}"/>
+  </joint>
 </robot>

Commit message: Import ROS simulation starting and map files

File: ros/src/clumsybot_description/urdf/clumsybot.urdf.xacro (robot description, xacro)
@@ -27,4 +27,9 @@
       <material name="metalic"/>
     </visual>
+    <collision>
+      <geometry>
+        <box size="${base_len} ${base_width + 2*hat_protuding} ${base_height + hat_height}"/>
+      </geometry>
+    </collision>
   </link>
   <link name="hat_link">

Commit message: Split simulation and rviz scripts, bot now visualizes in Gazebo

File: ros/src/clumsybot_description/urdf/clumsybot.urdf.xacro (robot description, xacro)
@@ -10,13 +10,6 @@
   <xacro:property name="wheel_width" value="0.007"/>
   <xacro:property name="wheel_clearance" value="0.005"/>
-  <material name="blue">
-    <color rgba="0 0 0.8 1"/>
-  </material>
-  <material name="metalic">
-    <color rgba="0.8 0.8 0.9 1"/>
-  </material>
-  <material name="wheel_color">
-    <color rgba="0.1 0.1 0.1 1"/>
-  </material>
+  <xacro:include filename="materials.xacro" />
+  <xacro:include filename="clumsybot.gazebo" />
   <link name="base_link">
     <visual>
@@ -32,5 +25,19 @@
       </geometry>
     </collision>
+    <inertial>
+      <origin xyz="0 0 ${base_height/2}" />
+      <mass value="1"/>
+      <inertia
+        ixx="1.0" ixy="0.0" ixz="0.0"
+        iyy="1.0" iyz="0.0"
+        izz="1.0"/>
+    </inertial>
   </link>
+  <link name="base_footprint"/>
+  <joint name="base_joint" type="fixed">
+    <parent link="base_footprint"/>
+    <child link="base_link"/>
+    <origin xyz="0.0 0.0 ${wheel_clearance}" rpy="0 0 0"/>
+  </joint>
   <link name="hat_link">
     <visual>
@@ -40,4 +47,12 @@
       <material name="blue"/>
     </visual>
+    <inertial>
+      <origin xyz="0 0 0" />
+      <mass value="1"/>
+      <inertia
+        ixx="1.0" ixy="0.0" ixz="0.0"
+        iyy="1.0" iyz="0.0"
+        izz="1.0"/>
+    </inertial>
   </link>
   <joint name="base_to_hat" type="fixed">
@@ -54,4 +69,12 @@
       <origin rpy="${PI/2} 0 0" />
     </visual>
+    <inertial>
+      <origin xyz="0 0 0" />
+      <mass value="0.1"/>
+      <inertia
+        ixx="1.0" ixy="0.0" ixz="0.0"
+        iyy="1.0" iyz="0.0"
+        izz="1.0"/>
+    </inertial>
   </link>
   <joint name="left_front_wheel_joint" type="continuous">
@@ -69,4 +92,12 @@
       <origin rpy="${PI/2} 0 0" />
     </visual>
+    <inertial>
+      <origin xyz="0 0 0" />
+      <mass value="0.1"/>
+      <inertia
+        ixx="1.0" ixy="0.0" ixz="0.0"
+        iyy="1.0" iyz="0.0"
+        izz="1.0"/>
+    </inertial>
   </link>
   <joint name="left_back_wheel_joint" type="continuous">
@@ -85,4 +116,12 @@
       <origin rpy="${PI/2} 0 0" />
     </visual>
+    <inertial>
+      <origin xyz="0 0 0" />
+      <mass value="0.1"/>
+      <inertia
+        ixx="1.0" ixy="0.0" ixz="0.0"
+        iyy="1.0" iyz="0.0"
+        izz="1.0"/>
+    </inertial>
   </link>
   <joint name="right_front_wheel_joint" type="continuous">
@@ -100,4 +139,12 @@
       <origin rpy="${PI/2} 0 0" />
     </visual>
+    <inertial>
+      <origin xyz="0 0 0" />
+      <mass value="0.1"/>
+      <inertia
+        ixx="1.0" ixy="0.0" ixz="0.0"
+        iyy="1.0" iyz="0.0"
+        izz="1.0"/>
+    </inertial>
   </link>
   <joint name="right_back_wheel_joint" type="continuous">

Commit message: Add differential drive ROS Gazebo simulation plugin, which isn't working as expected

File: ros/src/clumsybot_description/urdf/clumsybot.urdf.xacro (robot description, xacro)
@@ -21,4 +21,5 @@
     </visual>
     <collision>
+      <origin xyz="0 0 ${(base_height + hat_height)/2}" rpy="0 0 0" />
       <geometry>
         <box size="${base_len} ${base_width + 2*hat_protuding} ${base_height + hat_height}"/>
@@ -69,4 +70,10 @@
       <origin rpy="${PI/2} 0 0" />
     </visual>
+    <collision>
+      <geometry>
+        <cylinder length="${wheel_width}" radius="${wheel_radius}"/>
+      </geometry>
+      <origin rpy="${PI/2} 0 0" />
+    </collision>
     <inertial>
       <origin xyz="0 0 0" />
@@ -82,5 +89,5 @@
     <parent link="base_link"/>
     <child link="left_front_wheel"/>
-    <origin xyz="${-base_len/2 + wheel_radius} ${base_width/2} ${wheel_radius - wheel_clearance}"/>
+    <origin xyz="${-base_len/2 + wheel_radius} ${base_width/2 + wheel_width} ${wheel_radius - wheel_clearance}"/>
   </joint>
   <link name="left_back_wheel">
@@ -92,4 +99,10 @@
       <origin rpy="${PI/2} 0 0" />
     </visual>
+    <collision>
+      <geometry>
+        <cylinder length="${wheel_width}" radius="${wheel_radius}"/>
+      </geometry>
+      <origin rpy="${PI/2} 0 0" />
+    </collision>
     <inertial>
       <origin xyz="0 0 0" />
@@ -106,5 +119,5 @@
     <parent link="base_link"/>
     <child link="left_back_wheel"/>
-    <origin xyz="${base_len/2 - wheel_radius} ${base_width/2} ${wheel_radius - wheel_clearance}"/>
+    <origin xyz="${base_len/2 - wheel_radius} ${base_width/2 + wheel_width} ${wheel_radius - wheel_clearance}"/>
   </joint>
   <link name="right_front_wheel">
@@ -116,4 +129,10 @@
       <origin rpy="${PI/2} 0 0" />
     </visual>
+    <collision>
+      <geometry>
+        <cylinder length="${wheel_width}" radius="${wheel_radius}"/>
+      </geometry>
+      <origin rpy="${PI/2} 0 0" />
+    </collision>
     <inertial>
       <origin xyz="0 0 0" />
@@ -129,5 +148,5 @@
     <parent link="base_link"/>
     <child link="right_front_wheel"/>
-    <origin xyz="${-base_len/2 + wheel_radius} ${-base_width/2} ${wheel_radius - wheel_clearance}"/>
+    <origin xyz="${-base_len/2 + wheel_radius} ${-base_width/2 - wheel_width} ${wheel_radius - wheel_clearance}"/>
   </joint>
   <link name="right_back_wheel">
@@ -136,4 +155,10 @@
         <cylinder length="${wheel_width}" radius="${wheel_radius}"/>
       </geometry>
+      <collision>
+        <geometry>
+          <cylinder length="${wheel_width}" radius="${wheel_radius}"/>
+        </geometry>
+        <origin rpy="${PI/2} 0 0" />
+      </collision>
       <material name="wheel_color"/>
       <origin rpy="${PI/2} 0 0" />
@@ -153,5 +178,25 @@
     <parent link="base_link"/>
     <child link="right_back_wheel"/>
-    <origin xyz="${base_len/2 - wheel_radius} ${-base_width/2} ${wheel_radius - wheel_clearance}"/>
-  </joint>
+    <origin xyz="${base_len/2 - wheel_radius} ${-base_width/2 - wheel_width} ${wheel_radius - wheel_clearance}"/>
+  </joint>
+  <!-- <transmission name="left_wheel_transmission">
+    <type>transmission_interface/SimpleTransmission</type>
+    <joint name="left_front_wheel_joint">
+      <hardwareInterface>hardware_interface/VelocityJointInterface</hardwareInterface>
+    </joint>
+    <actuator name="left_wheel_actuator">
+      <mechanicalReduction>7</mechanicalReduction>
+      <hardwareInterface>VelocityJointInterface</hardwareInterface>
+    </actuator>
+  </transmission>
+  <transmission name="right_wheel_transmission">
+    <type>transmission_interface/SimpleTransmission</type>
+    <joint name="right_front_wheel_joint">
+      <hardwareInterface>hardware_interface/VelocityJointInterface</hardwareInterface>
+    </joint>
+    <actuator name="right_wheel_actuator">
+      <mechanicalReduction>7</mechanicalReduction>
+      <hardwareInterface>VelocityJointInterface</hardwareInterface>
+    </actuator>
+  </transmission> -->
 </robot>

Commit message: Fix ROS Gazebo simulation plugin for differential wheel movement. Now bot is nicely movable

File: ros/src/clumsybot_description/urdf/clumsybot.urdf.xacro (robot description, xacro)
@@ -28,5 +28,5 @@
     <inertial>
       <origin xyz="0 0 ${base_height/2}" />
-      <mass value="1"/>
+      <mass value="2"/>
       <inertia
         ixx="1.0" ixy="0.0" ixz="0.0"
@@ -49,6 +49,5 @@
     </visual>
     <inertial>
-      <origin xyz="0 0 0" />
-      <mass value="1"/>
+      <mass value="0.5"/>
       <inertia
         ixx="1.0" ixy="0.0" ixz="0.0"
@@ -77,10 +76,9 @@
     </collision>
     <inertial>
-      <origin xyz="0 0 0" />
-      <mass value="0.1"/>
+      <mass value="0.01"/>
       <inertia
-        ixx="1.0" ixy="0.0" ixz="0.0"
-        iyy="1.0" iyz="0.0"
-        izz="1.0"/>
+        ixx="1.0e-5" ixy="0.0" ixz="0.0"
+        iyy="1.0e-5" iyz="0.0"
+        izz="1.0e-5"/>
     </inertial>
   </link>
@@ -89,5 +87,5 @@
     <parent link="base_link"/>
     <child link="left_front_wheel"/>
-    <origin xyz="${-base_len/2 + wheel_radius} ${base_width/2 + wheel_width} ${wheel_radius - wheel_clearance}"/>
+    <origin xyz="${-base_len/2 + wheel_radius} ${base_width/2} ${wheel_radius - wheel_clearance}"/>
   </joint>
   <link name="left_back_wheel">
@@ -106,10 +104,9 @@
     </collision>
     <inertial>
-      <origin xyz="0 0 0" />
-      <mass value="0.1"/>
+      <mass value="0.01"/>
       <inertia
-        ixx="1.0" ixy="0.0" ixz="0.0"
-        iyy="1.0" iyz="0.0"
-        izz="1.0"/>
+        ixx="1.0e-5" ixy="0.0" ixz="0.0"
+        iyy="1.0e-5" iyz="0.0"
+        izz="1.0e-5"/>
     </inertial>
   </link>
@@ -119,5 +116,5 @@
     <parent link="base_link"/>
     <child link="left_back_wheel"/>
-    <origin xyz="${base_len/2 - wheel_radius} ${base_width/2 + wheel_width} ${wheel_radius - wheel_clearance}"/>
+    <origin xyz="${base_len/2 - wheel_radius} ${base_width/2} ${wheel_radius - wheel_clearance}"/>
   </joint>
   <link name="right_front_wheel">
@@ -136,10 +133,9 @@
     </collision>
     <inertial>
-      <origin xyz="0 0 0" />
-      <mass value="0.1"/>
+      <mass value="0.01"/>
       <inertia
-        ixx="1.0" ixy="0.0" ixz="0.0"
-        iyy="1.0" iyz="0.0"
-        izz="1.0"/>
+        ixx="1.0e-5" ixy="0.0" ixz="0.0"
+        iyy="1.0e-5" iyz="0.0"
+        izz="1.0e-5"/>
     </inertial>
   </link>
@@ -148,5 +144,5 @@
     <parent link="base_link"/>
     <child link="right_front_wheel"/>
-    <origin xyz="${-base_len/2 + wheel_radius} ${-base_width/2 - wheel_width} ${wheel_radius - wheel_clearance}"/>
+    <origin xyz="${-base_len/2 + wheel_radius} ${-base_width/2} ${wheel_radius - wheel_clearance}"/>
   </joint>
   <link name="right_back_wheel">
@@ -155,20 +151,19 @@
         <cylinder length="${wheel_width}" radius="${wheel_radius}"/>
       </geometry>
-      <collision>
-        <geometry>
-          <cylinder length="${wheel_width}" radius="${wheel_radius}"/>
-        </geometry>
-        <origin rpy="${PI/2} 0 0" />
-      </collision>
+      <origin rpy="${PI/2} 0 0" />
       <material name="wheel_color"/>
+    </visual>
+    <collision>
+      <geometry>
+        <cylinder length="${wheel_width}" radius="${wheel_radius}"/>
+      </geometry>
       <origin rpy="${PI/2} 0 0" />
-    </visual>
+    </collision>
     <inertial>
-      <origin xyz="0 0 0" />
-      <mass value="0.1"/>
+      <mass value="0.01"/>
       <inertia
-        ixx="1.0" ixy="0.0" ixz="0.0"
-        iyy="1.0" iyz="0.0"
-        izz="1.0"/>
+        ixx="1.0e-5" ixy="0.0" ixz="0.0"
+        iyy="1.0e-5" iyz="0.0"
+        izz="1.0e-5"/>
     </inertial>
   </link>
@@ -178,5 +173,5 @@
     <parent link="base_link"/>
     <child link="right_back_wheel"/>
-    <origin xyz="${base_len/2 - wheel_radius} ${-base_width/2 - wheel_width} ${wheel_radius - wheel_clearance}"/>
+    <origin xyz="${base_len/2 - wheel_radius} ${-base_width/2} ${wheel_radius - wheel_clearance}"/>
   </joint>
   <!-- <transmission name="left_wheel_transmission">

Commit message: Link ROS Gazebo diff drive odometry output to RViz

File: ros/src/clumsybot_description/urdf/clumsybot.urdf.xacro (robot description, xacro)
@@ -175,4 +175,23 @@
     <origin xyz="${base_len/2 - wheel_radius} ${-base_width/2} ${wheel_radius - wheel_clearance}"/>
   </joint>
+  <!-- <link name="kinect_link">
+    <visual>
+      <geometry>
+        <box size="0.02 0.18 0.02"/>
+      </geometry>
+    </visual>
+    <inertial>
+      <mass value="0.5"/>
+      <inertia
+        ixx="1.0" ixy="0.0" ixz="0.0"
+        iyy="1.0" iyz="0.0"
+        izz="1.0"/>
+    </inertial>
+  </link>
+  <joint name="kinect_to_hat_joint" type="fixed">
+    <parent link="hat_link"/>
+    <child link="kinect_link"/>
+    <origin xyz="0 0 ${hat_height+0.03}" />
+  </joint> -->
   <!-- <transmission name="left_wheel_transmission">
     <type>transmission_interface/SimpleTransmission</type>

Commit message: Tidy up ROS URDF, Gazebo Kinect plugin still refuses to work (probably as it does not exist for foxy ros version)

File: ros/src/clumsybot_description/urdf/clumsybot.urdf.xacro (robot description, xacro)
@@ -30,7 +30,7 @@
       <mass value="2"/>
       <inertia
-        ixx="1.0" ixy="0.0" ixz="0.0"
-        iyy="1.0" iyz="0.0"
-        izz="1.0"/>
+        ixx="1.0e-3" ixy="0.0" ixz="0.0"
+        iyy="1.0e-3" iyz="0.0"
+        izz="1.0e-3"/>
     </inertial>
   </link>
@@ -51,7 +51,7 @@
       <mass value="0.5"/>
       <inertia
-        ixx="1.0" ixy="0.0" ixz="0.0"
-        iyy="1.0" iyz="0.0"
-        izz="1.0"/>
+        ixx="0" ixy="0.0" ixz="0.0"
+        iyy="0" iyz="0.0"
+        izz="0"/>
     </inertial>
   </link>
@@ -175,23 +175,17 @@
     <origin xyz="${base_len/2 - wheel_radius} ${-base_width/2} ${wheel_radius - wheel_clearance}"/>
   </joint>
-  <!-- <link name="kinect_link">
-    <visual>
-      <geometry>
-        <box size="0.02 0.18 0.02"/>
-      </geometry>
-    </visual>
-    <inertial>
-      <mass value="0.5"/>
-      <inertia
-        ixx="1.0" ixy="0.0" ixz="0.0"
-        iyy="1.0" iyz="0.0"
-        izz="1.0"/>
-    </inertial>
-  </link>
+  <xacro:include filename="sensor/kinect/kinect.urdf.xacro"/>
+  <xacro:kinect_cam name="kinect"/>
   <joint name="kinect_to_hat_joint" type="fixed">
     <parent link="hat_link"/>
     <child link="kinect_link"/>
     <origin xyz="0 0 ${hat_height+0.03}" />
-  </joint> -->
+  </joint>
+  <link name="kinect_rgb_optical_frame"/>
+  <joint name="rgb_kinect_joint" type="fixed">
+    <origin rpy="${PI/2} ${PI} ${PI/2}"/>
+    <parent link="kinect_link"/>
+    <child link="kinect_rgb_optical_frame"/>
+  </joint>
   <!-- <transmission name="left_wheel_transmission">
     <type>transmission_interface/SimpleTransmission</type>

Commit message: Add ROS Gazebo proximity sensor to bot

File: ros/src/clumsybot_description/urdf/clumsybot.urdf.xacro (robot description, xacro)
@@ -175,5 +175,5 @@
     <origin xyz="${base_len/2 - wheel_radius} ${-base_width/2} ${wheel_radius - wheel_clearance}"/>
   </joint>
-  <xacro:include filename="sensor/kinect/kinect.urdf.xacro"/>
+  <!-- <xacro:include filename="sensor/kinect/kinect.urdf.xacro"/>
   <xacro:kinect_cam name="kinect"/>
   <joint name="kinect_to_hat_joint" type="fixed">
@@ -187,5 +187,7 @@
     <parent link="kinect_link"/>
     <child link="kinect_rgb_optical_frame"/>
-  </joint>
+  </joint> -->
+  <xacro:include filename="sensor/proximity_sensor.urdf.xacro"/>
+  <xacro:proximity_sensor group="proximity" range_max="2.5" name="proxsense" xyz="0.08 0 0" rpy="0 0 0"/>
   <!-- <transmission name="left_wheel_transmission">
     <type>transmission_interface/SimpleTransmission</type>

Commit message: Import all ROS related untracked files

File: ros/src/clumsybot_description/urdf/clumsybot.urdf.xacro (robot description, xacro)
@@ -175,9 +175,9 @@
     <origin xyz="${base_len/2 - wheel_radius} ${-base_width/2} ${wheel_radius - wheel_clearance}"/>
   </joint>
-  <!-- <xacro:include filename="sensor/kinect/kinect.urdf.xacro"/>
-  <xacro:kinect_cam name="kinect"/>
+  <xacro:include filename="sensor/kinect/kinect.urdf.xacro"/>
+  <xacro:kinect_cam name="camera"/>
   <joint name="kinect_to_hat_joint" type="fixed">
     <parent link="hat_link"/>
-    <child link="kinect_link"/>
+    <child link="camera_link"/>
     <origin xyz="0 0 ${hat_height+0.03}" />
   </joint>
@@ -185,7 +185,7 @@
   <joint name="rgb_kinect_joint" type="fixed">
     <origin rpy="${PI/2} ${PI} ${PI/2}"/>
-    <parent link="kinect_link"/>
+    <parent link="camera_link"/>
     <child link="kinect_rgb_optical_frame"/>
-  </joint> -->
+  </joint>
   <xacro:include filename="sensor/proximity_sensor.urdf.xacro"/>
   <xacro:proximity_sensor group="proximity" range_max="2.5" name="proxsense" xyz="0.08 0 0" rpy="0 0 0"/>
